File: pcb/ai_breakout_ads1115.brd (EAGLE design)
At the start: 15.2 x 12.7 mm, 13 parts, among them J1 1X05, J2 1X05, U1 ADS1115

Commit message: major changes
Parts:
- J2: value 1X05 -> 1X05NOFIRST; device Ai_Connectors:1X05 -> Ai_Connectors:1X05-NOFIRST
- moved U$2 3.56 mm to (5.08, 0.51)
- moved R2 3.05 mm to (7.49, 1.70)
- moved R4 1.54 mm to (10.5, 1.70)
- moved R3 1.54 mm to (9.02, 1.70)
- moved C1 0.20 mm to (4.45, 1.70)
- moved FB1 0.20 mm to (5.82, 1.70)
- moved FB2 0.13 mm to (5.21, 10.4)
- renumbered JS1 to 0X48
Connections:
- net ADDR: now also R3.1; no longer R4.1
- net ALERT: now also R2.1; no longer R3.1
- net SDA: now also R4.1; no longer R2.1
Other:
- board text added: "16-Bit ADC 4-Channel (ADS1115)"
- board text added: "I2C Address: 0x49 Default 0x48 w Solder"
- board text added: "https://acrobotic.com"
- board text added: "v1.0"
- board text removed: "ADS115 Analog-Digital Converter"
