File: pcb/ai_breakout_ads1115.sch (EAGLE design)
At the start: 13 parts, among them J1 1X05, J2 1X05, U1 ADS1115

Commit message: major changes
Parts:
- J2: value 1X05 -> 1X05NOFIRST; device Ai_Connectors:1X05 -> Ai_Connectors:1X05NOFIRST
- renumbered JS1 to 0X48
Connections:
- net ADDR: now also R3.1; no longer R4.1
- net ALERT: now also R2.1; no longer R3.1
- net SDA: now also R4.1; no longer R2.1
Other:
- moved on the sheet: R2, R3, R4
Changed lines of the file:
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@@
 <part name="U1" library="Ai_IC" deviceset="ADS1115" device="" value="ADS1115"/>
 <part name="FRAME1" library="Ai_Miscellany" deviceset="FRAME-LETTER" device="">
-<attribute name="AUTHOR" value="A.I. HERMOSAURUS"/>
+<attribute name="AUTHOR" value="A.I. Jeffrey Hermosura"/>
 <attribute name="REV" value="1.0"/>
 </part>
@@
 <part name="VCC1" library="Ai_Power" deviceset="VDD" device=""/>
 <part name="R1" library="Ai_Passives" deviceset="RES" device="0603" value="10K"/>
+<part name="R4" library="Ai_Passives" deviceset="RES" device="0603" value="10K"/>
 <part name="R2" library="Ai_Passives" deviceset="RES" device="0603" value="10K"/>
+<part name="VCC2" library="Ai_Power" deviceset="VDD" device=""/>
+<part name="0X48" library="Ai_Connectors" deviceset="1X02-SJ-NO" device=""/>
+<part name="C2" library="Ai_Passives" deviceset="CAP" device="0603" value="100nF"/>
 <part name="R3" library="Ai_Passives" deviceset="RES" device="0603" value="10K"/>
-<part name="VCC2" library="Ai_Power" deviceset="VDD" device=""/>
-<part name="JS1" library="Ai_Connectors" deviceset="1X02-SJ-NO" device=""/>
-<part name="C2" library="Ai_Passives" deviceset="CAP" device="0603" value="100nF"/>
-<part name="R4" library="Ai_Passives" deviceset="RES" device="0603" value="10K"/>
-<part name="J2" library="Ai_Connectors" deviceset="1X05" device=""/>
+<part name="J2" library="Ai_Connectors" deviceset="1X05" device="NOFIRST" value="1X05NOFIRST"/>
 <part name="J1" library="Ai_Connectors" deviceset="1X05" device=""/>
 <part name="C1" library="Ai_Passives" deviceset="CAP" device="0603" value="10uF"/>
@@
 <instance part="VCC1" gate="G$1" x="165.1" y="123.19"/>
 <instance part="R1" gate="G$1" x="193.04" y="111.76" rot="R90"/>
-<instance part="R2" gate="G$1" x="198.12" y="111.76" rot="R90"/>
-<instance part="R3" gate="G$1" x="182.88" y="111.76" rot="R90"/>
+<instance part="R4" gate="G$1" x="198.12" y="111.76" rot="R90"/>
+<instance part="R2" gate="G$1" x="182.88" y="111.76" rot="R90"/>
 <instance part="VCC2" gate="G$1" x="193.04" y="123.19"/>
-<instance part="JS1" gate="1" x="203.2" y="91.44" rot="R270"/>
+<instance part="0X48" gate="1" x="203.2" y="91.44" rot="R270"/>
 <instance part="C2" gate="G$1" x="111.76" y="109.22" rot="R180"/>
-<instance part="R4" gate="G$1" x="187.96" y="111.76" rot="R90"/>
+<instance part="R3" gate="G$1" x="187.96" y="111.76" rot="R90"/>
 <instance part="J2" gate="G$1" x="50.8" y="81.28"/>
 <instance part="J1" gate="G$1" x="50.8" y="101.6"/>
@@
 </segment>
 <segment>
-<pinref part="JS1" gate="1" pin="2"/>
+<pinref part="0X48" gate="1" pin="2"/>
 <pinref part="GND2" gate="GND" pin="GND"/>
 <wire x1="203.2" y1="81.28" x2="203.2" y2="86.36" width="0.1524" layer="91"/>
@@
 <wire x1="176.53" y1="104.14" x2="182.88" y2="104.14" width="0.1524" layer="91"/>
 <wire x1="182.88" y1="104.14" x2="182.88" y2="106.68" width="0.1524" layer="91"/>
-<pinref part="R3" gate="G$1" pin="1"/>
+<pinref part="R2" gate="G$1" pin="1"/>
 <wire x1="182.88" y1="104.14" x2="205.74" y2="104.14" width="0.1524" layer="91"/>
 <junction x="182.88" y="104.14"/>
@@
 <wire x1="187.96" y1="99.06" x2="203.2" y2="99.06" width="0.1524" layer="91"/>
 <wire x1="203.2" y1="99.06" x2="203.2" y2="96.52" width="0.1524" layer="91"/>
-<pinref part="JS1" gate="1" pin="1"/>
-<pinref part="R4" gate="G$1" pin="1"/>
+<pinref part="0X48" gate="1" pin="1"/>
+<pinref part="R3" gate="G$1" pin="1"/>
 <wire x1="187.96" y1="99.06" x2="187.96" y2="106.68" width="0.1524" layer="91"/>
 <wire x1="203.2" y1="99.06" x2="205.74" y2="99.06" width="0.1524" layer="91"/>
@@
 <wire x1="176.53" y1="88.9" x2="198.12" y2="88.9" width="0.1524" layer="91"/>
 <wire x1="198.12" y1="88.9" x2="198.12" y2="106.68" width="0.1524" layer="91"/>
-<pinref part="R2" gate="G$1" pin="1"/>
+<pinref part="R4" gate="G$1" pin="1"/>
 </segment>
 </net>
@@
 <segment>
 <wire x1="146.05" y1="119.38" x2="165.1" y2="119.38" width="0.1524" layer="91"/>
-<pinref part="R3" gate="G$1" pin="2"/>
+<pinref part="R2" gate="G$1" pin="2"/>
 <wire x1="165.1" y1="119.38" x2="182.88" y2="119.38" width="0.1524" layer="91"/>
 <wire x1="182.88" y1="119.38" x2="182.88" y2="116.84" width="0.1524" layer="91"/>
@@
 </segment>
 <segment>
-<pinref part="R4" gate="G$1" pin="2"/>
+<pinref part="R3" gate="G$1" pin="2"/>
 <wire x1="187.96" y1="116.84" x2="187.96" y2="123.19" width="0.1524" layer="91"/>
 <pinref part="VCC3" gate="G$1" pin="VDD"/>
@@
 <segment>
 <pinref part="VCC6" gate="G$1" pin="VDD"/>
-<pinref part="R2" gate="G$1" pin="2"/>
+<pinref part="R4" gate="G$1" pin="2"/>
 <wire x1="198.12" y1="123.19" x2="198.12" y2="116.84" width="0.1524" layer="91"/>
 </segment>
